File: hw/sch_pcb/TFHT02.kicad_pcb (KiCad board)
At the start: 2 copper layers, 30 x 15 mm, 20 parts, among them J1 SM04B-GHS-TB, J2 SM04B-GHS-TB, M1 M3, M2 M3, M3 M3, M4 M3, M5 M3, M6 M3, U2 SHT4x, U3 MIC5504-3.3YM5

Commit message: Improved layout and geometry.
Parts:
- moved U2 0.35 mm to (159.3, 112.6)
- moved C1 0.31 mm to (145.8, 115.9)
- moved U3 0.30 mm to (142.9, 116.1)
- moved C3 0.07 mm to (139.8, 116.0)
Routing:
- net GND: track 42.1 -> 40.4 mm, vias 19 -> 18
- net +3V3: track 25.8 -> 24.9 mm
- net +5V: track 22.9 -> 23.4 mm
- net /SCL: track 29.3 -> 29.5 mm, vias 2 -> 1
Other:
- outline, holes or cut-outs redrawn
- rule pad_to_mask_clearance: 0.2 -> 0.05
